File: apppd.kicad_pcb (KiCad board)
At the start: 2 copper layers, 59 parts, among them J1 Conn_SWD, J2 APPPD Connector, J4 2601-1102, J5 USB_C_Receptacle_USB2.0_16P, Q1 AO3400A, Q2 AO3400A, SW1 NRST, SW2 BOOT0, U1 AP2112K-3.3, U2 STM32F072CBTx, U3 USBLC6-2SC6, U4 TCAN337, U5 SN74LVC2G14DBVR

Commit message: update
Parts:
- moved C10 68.1 mm to (25.8, 25.5)
- moved SW1 55.0 mm to (19.5, 22.2)
- moved SW2 52.5 mm to (19.2, 29.2)
- moved LED1 48.7 mm to (33.2, 36.5), turned to 90 degrees
- moved R13 47.4 mm to (83.2, 60.2)
- moved R17 47.3 mm to (88.8, 56.8)
- moved R18 47.3 mm to (88.8, 59.7)
- moved R8 46.5 mm to (83.5, 56.8)
- moved FB1 41.8 mm to (46.0, 36.5)
- moved C6 39.7 mm to (53.8, 39.5)
- moved C11 39.7 mm to (58.6, 42.5)
- moved C4 39.7 mm to (48.9, 45.5)
- moved C5 39.7 mm to (53.8, 36.5)
- moved C7 39.7 mm to (53.8, 42.5)
- moved C8 39.7 mm to (53.8, 45.5)
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
Commit message: Voltage shift for apps and tps sensors, 3v3 compatability
Parts:
- moved R1 80.3 mm to (43.5, 107.5)
- moved SW1 79.2 mm to (43.5, 97.8)
- moved SW2 79.1 mm to (43.5, 104.5)
- moved C10 77.1 mm to (43.5, 100.5)
Changed lines of the file:
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@@
 	(footprint "Capacitor_SMD:C_0805_2012Metric_Pad1.18x1.45mm_HandSolder"
 		(layer "F.Cu")
-		(at 25.75 25.5)
+		(at 43.5 100.5)
 		(descr "Capacitor SMD 0805 (2012 Metric), square (rectangular) end terminal, IPC-7351 nominal with elongated pad for handsoldering. (Body size source: IPC-SM-782 page 76, https://www.pcb-3d.com/wordpress/wp-content/uploads/ipc-sm-782a_amendment_1_and_2.pdf, https://docs.google.com/spreadsheets/d/1BsfQQcO9C6DZCsRaXUlFlo91Tg2WpOkGARC1WS5S8t0/edit?usp=sharing)")
 		(tags "capacitor handsolder")
 		(property "Reference" "C10"
-			(at 0 -1.68 0)
+			(at 3.5 0 0)
 			(layer "F.SilkS")
 			(effects
@@
 	(footprint "apppd:SW-SMD_L3.9-W3.0-P4.45"
 		(layer "F.Cu")
-		(at 19.25 29.25)
+		(at 43.5 104.5)
 		(property "Reference" "SW2"
 			(at 0 -2.25 0)
@@
 				(font
 					(size 1.27 1.27)
+					(thickness 0.15)
 				)
 			)
@@
 		)
 		(embedded_fonts no)
-		(model "C:/Users/chith/Documents/KiCad/easyeda2kicad/easyeda2kicad.3dshapes/SW-SMD_L3.9-W2.9-H2.0-LS4.8.wrl"
+		(model "${KIPRJMOD}/library/3d/SW-SMD_L3.9-W2.9-H2.0-LS4.8.step"
 			(offset
 				(xyz 0 0 0)
@@
 	(footprint "apppd:SW-SMD_L3.9-W3.0-P4.45"
 		(layer "F.Cu")
-		(at 19.5 22.25)
+		(at 43.5 97.75)
 		(property "Reference" "SW1"
 			(at 0 -2.25 0)
@@
 				(font
 					(size 1.27 1.27)
+					(thickness 0.15)
 				)
 			)
@@
 		)
 		(embedded_fonts no)
-		(model "C:/Users/chith/Documents/KiCad/easyeda2kicad/easyeda2kicad.3dshapes/SW-SMD_L3.9-W2.9-H2.0-LS4.8.wrl"
+		(model "${KIPRJMOD}/library/3d/SW-SMD_L3.9-W2.9-H2.0-LS4.8.step"
 			(offset
 				(xyz 0 0 0)
@@
 	(footprint "Resistor_SMD:R_0805_2012Metric_Pad1.20x1.40mm_HandSolder"
 		(layer "F.Cu")
-		(at 25.5 29.25)
+		(at 43.5 107.5)
 		(descr "Resistor SMD 0805 (2012 Metric), square (rectangular) end terminal, IPC-7351 nominal with elongated pad for handsoldering. (Body size source: IPC-SM-782 page 72, https://www.pcb-3d.com/wordpress/wp-content/uploads/ipc-sm-782a_amendment_1_and_2.pdf)")
 		(tags "resistor handsolder")
 		(property "Reference" "R1"
-			(at 0 -1.65 0)
+			(at 3 0 0)
 			(layer "F.SilkS")
 			(effects
@@
 				(font
 					(size 1.27 1.27)
+					(thickness 0.15)
 				)
 			)
@@
 		)
 		(embedded_fonts no)
-		(model "C:/Users/chith/Documents/KiCad/easyeda2kicad/easyeda2kicad.3dshapes/USB-C-SMD_TYPE-C-6PIN-2MD-073.wrl"
+		(model "${KIPRJMOD}/library/3d/USB-C-SMD_TYPE-C-6PIN-2MD-073.step"
 			(offset
 				(xyz 0 0 0)
@@
 				(font
 					(size 1.27 1.27)
+					(thickness 0.15)
 				)
 			)

Commit message: Fixed ground and small changes
Parts:
- removed R13: 150, Resistor_SMD:R_0805_2012Metric_Pad1.20x1.40mm_HandSolder
- removed R16, R17: 150k, Resistor_SMD:R_0805_2012Metric_Pad1.20x1.40mm_HandSolder
- removed R18: 100k, Resistor_SMD:R_0805_2012Metric_Pad1.20x1.40mm_HandSolder
- added C13: 8pF, Capacitor_SMD:C_0805_2012Metric_Pad1.18x1.45mm_HandSolder, F.Cu at (107.2, 67.5)
- added C14: 8pF, Capacitor_SMD:C_0805_2012Metric_Pad1.18x1.45mm_HandSolder, F.Cu at (107.2, 70.5)
- added C15: 10uF, Capacitor_SMD:C_0805_2012Metric_Pad1.18x1.45mm_HandSolder, F.Cu at (107.2, 73.5)
- added C16: 220nF, Capacitor_SMD:C_0805_2012Metric_Pad1.18x1.45mm_HandSolder, F.Cu at (107.2, 76.5)
- added C17: 1uF, Capacitor_SMD:C_0805_2012Metric_Pad1.18x1.45mm_HandSolder, F.Cu at (107.2, 79.6)
- added C18: 100nF, Capacitor_SMD:C_0805_2012Metric_Pad1.18x1.45mm_HandSolder, F.Cu at (112.0, 64.5)
- added C19: 22uF, Capacitor_SMD:C_0805_2012Metric_Pad1.18x1.45mm_HandSolder, F.Cu at (112.0, 67.5)
- added C20: 22uF, Capacitor_SMD:C_0805_2012Metric_Pad1.18x1.45mm_HandSolder, F.Cu at (112.0, 70.5)
- added C21: 1uF, Capacitor_SMD:C_0805_2012Metric_Pad1.18x1.45mm_HandSolder, F.Cu at (112.0, 73.5)
- added C22: 1uF, Capacitor_SMD:C_0805_2012Metric_Pad1.18x1.45mm_HandSolder, F.Cu at (112.0, 76.5)
- added C23: 1uF, Capacitor_SMD:C_0805_2012Metric_Pad1.18x1.45mm_HandSolder, F.Cu at (112.0, 79.6)
- added C24: 10uF, Capacitor_SMD:C_0805_2012Metric_Pad1.18x1.45mm_HandSolder, F.Cu at (116.8, 64.5)
- added C25: 1uF, Capacitor_SMD:C_0805_2012Metric_Pad1.18x1.45mm_HandSolder, F.Cu at (116.8, 67.5)
- added C26: 100nF, Capacitor_SMD:C_0805_2012Metric_Pad1.18x1.45mm_HandSolder, F.Cu at (116.8, 70.5)
- added C27: 100nF, Capacitor_SMD:C_0805_2012Metric_Pad1.18x1.45mm_HandSolder, F.Cu at (116.8, 73.5)
- added D10: PMEG2010BER, Diode_SMD:Nexperia_CFP3_SOD-123W, F.Cu at (88.6, 85.3)
- added D11: PMEG2010BER, Diode_SMD:Nexperia_CFP3_SOD-123W, F.Cu at (88.6, 88.5)
- added D12: SZESD9B5.0ST5G, Diode_SMD:D_SOD-923, F.Cu at (122.7, 87.9)
- added D7: S1B-13-F, apppd:S1B-13-F, F.Cu at (117.3, 83.3)
- added D8: S1B-13-F, apppd:S1B-13-F, F.Cu at (117.3, 87.9)
- added D9: SZESD9B5.0ST5G, Diode_SMD:D_SOD-923, F.Cu at (122.7, 85.9)
- added L1: 8.2uH, 86m, Inductor_SMD:L_Vishay_IHLP-1616, F.Cu at (94.9, 86.5)
- added Q3: PMV100EPA, Package_TO_SOT_SMD:TSOT-23_HandSoldering, F.Cu at (108.2, 96.7)
- added R21: 1k, Resistor_SMD:R_0805_2012Metric_Pad1.20x1.40mm_HandSolder, F.Cu at (88.1, 76.3)
- added R22: 1k, Resistor_SMD:R_0805_2012Metric_Pad1.20x1.40mm_HandSolder, F.Cu at (88.1, 79.2)
- added R26: 150, Resistor_SMD:R_0805_2012Metric_Pad1.20x1.40mm_HandSolder, F.Cu at (88.1, 82.2)
- added R27: 150, Resistor_SMD:R_0805_2012Metric_Pad1.20x1.40mm_HandSolder, F.Cu at (92.9, 64.5)
- added R28: 150, Resistor_SMD:R_0805_2012Metric_Pad1.20x1.40mm_HandSolder, F.Cu at (92.9, 67.4)
- added R29: 100k, Resistor_SMD:R_0805_2012Metric_Pad1.20x1.40mm_HandSolder, F.Cu at (92.9, 70.4)
- added R30: 100k, Resistor_SMD:R_0805_2012Metric_Pad1.20x1.40mm_HandSolder, F.Cu at (92.9, 73.3)
- added R31: 100k, Resistor_SMD:R_0805_2012Metric_Pad1.20x1.40mm_HandSolder, F.Cu at (92.9, 76.3)
- added R32: 100k, Resistor_SMD:R_0805_2012Metric_Pad1.20x1.40mm_HandSolder, F.Cu at (92.9, 79.2)
- added R33: 150, Resistor_SMD:R_0805_2012Metric_Pad1.20x1.40mm_HandSolder, F.Cu at (92.9, 82.2)
- added R34: 100k, Resistor_SMD:R_0805_2012Metric_Pad1.20x1.40mm_HandSolder, F.Cu at (97.6, 64.5)
- added R35: 100k, Resistor_SMD:R_0805_2012Metric_Pad1.20x1.40mm_HandSolder, F.Cu at (97.6, 67.4)
- added R36: 100k, Resistor_SMD:R_0805_2012Metric_Pad1.20x1.40mm_HandSolder, F.Cu at (97.6, 70.4)
- added R37: 100k, Resistor_SMD:R_0805_2012Metric_Pad1.20x1.40mm_HandSolder, F.Cu at (97.6, 73.3)
- added R38: 300k, Resistor_SMD:R_0805_2012Metric_Pad1.20x1.40mm_HandSolder, F.Cu at (97.6, 76.3)
- added R39: 300k, Resistor_SMD:R_0805_2012Metric_Pad1.20x1.40mm_HandSolder, F.Cu at (97.6, 79.2)
- added R40: 300k, Resistor_SMD:R_0805_2012Metric_Pad1.20x1.40mm_HandSolder, F.Cu at (97.6, 82.2)
- added R41: 300k, Resistor_SMD:R_0805_2012Metric_Pad1.20x1.40mm_HandSolder, F.Cu at (102.4, 64.5)
- added R46: 5.49k, Resistor_SMD:R_0805_2012Metric_Pad1.20x1.40mm_HandSolder, F.Cu at (102.4, 67.4)
- added R47: 5.49k, Resistor_SMD:R_0805_2012Metric_Pad1.20x1.40mm_HandSolder, F.Cu at (102.4, 70.4)
- added R48: 5.49k, Resistor_SMD:R_0805_2012Metric_Pad1.20x1.40mm_HandSolder, F.Cu at (102.4, 73.3)
- added R49: 5.49k, Resistor_SMD:R_0805_2012Metric_Pad1.20x1.40mm_HandSolder, F.Cu at (102.4, 76.3)
- added TP1: TPS1, TestPoint:TestPoint_Keystone_5000-5004_Miniature, F.Cu at (121.4, 65.2)
- added TP2: TPS2, TestPoint:TestPoint_Keystone_5000-5004_Miniature, F.Cu at (121.4, 69.5)
- added TP3: BPS, TestPoint:TestPoint_Keystone_5000-5004_Miniature, F.Cu at (121.4, 73.9)
- added TP4: BPS, TestPoint:TestPoint_Keystone_5000-5004_Miniature, F.Cu at (121.4, 78.2)
- added U6: LMR33610ADDAR, Package_SO:Texas_HSOP-8-1EP_3.9x4.9mm_P1.27mm_ThermalVias, F.Cu at (117.5, 93.5)
- added U7: TLV9062xD, Package_SO:SOIC-8_3.9x4.9mm_P1.27mm, F.Cu at (109.0, 91.0)
- added Y1: ABM8AIG-24.000MHz-8-2Z-T, apppd:ABM8AIG-24.000MHZ-8-2Z-T, F.Cu at (101.4, 86.2)
- C4: value 100nF -> 1uF
- D1: value LED -> BZT52-C15S-AU_R1_000A1; footprint apppd:AP2012EC -> Diode_SMD:D_SOD-323_HandSoldering
- D2: value LED -> SMBJ26A; footprint apppd:AP2012EC -> Diode_SMD:D_SMA-SMB_Universal_Handsoldering
- D3, D5: value S1B-13-F -> LED; footprint apppd:S1B-13-F -> apppd:AP2012EC
- D4, D6: value S1B-13-F -> SZESD9B5.0ST5G; footprint apppd:S1B-13-F -> Diode_SMD:D_SOD-923
- F1: value 100mA Polyfuse -> 300mA Polyfuse
- R10, R11, R15, R9: value 150k -> 100k
- R12: value 100k -> 24.9k
- R8: value 150 -> 10K
- U5: value SN74LVC2G14DBVR -> TLV9062xD; footprint apppd:SN74LVC2G14DBVR -> Package_SO:SOIC-8_3.9x4.9mm_P1.27mm
- moved D4 64.3 mm to (122.7, 82.0)
- moved D6 62.4 mm to (122.7, 84.0)
- moved C4 61.2 mm to (107.2, 64.5)
- moved R10 51.4 mm to (88.1, 67.4)
- moved R11 51.4 mm to (88.1, 70.4)
- moved R12 51.4 mm to (88.1, 73.3)
- moved D3 43.5 mm to (88.3, 91.6)
- moved U5 39.2 mm to (109.0, 84.4)
- moved D5 38.8 mm to (88.3, 94.4)
- moved D1 33.4 mm to (93.9, 96.3)
- moved D2 27.2 mm to (96.9, 92.0)
- moved R8 9.00 mm to (88.1, 64.5)
Connections:
- net Net-(U2-VDDA) renamed /VDDA
- C4 pad 1: GND -> Net-(U5A-+)
- C4 pad 2: +3V3 -> Earth
- D1 pad 1: GND -> /buckIN
- D2 pad 1: GND -> +12V
- D2 pad 2: Net-(D2-A) -> GND
- D3 pad 1: IGN_OUT -> Net-(D3-K)
- D3 pad 2: GND -> +12V
- D4 pad 1: +12V -> Earth
- D4 pad 2: IGN_OUT -> APPS1_RAW
- D5 pad 1: ETB_OUT -> Net-(D5-K)
- D5 pad 2: GND -> +12V
- D6 pad 1: +12V -> Earth
- D6 pad 2: ETB_OUT -> APPS2_RAW
- F1 pad 1: VBUS -> +5V
- J2 pad 1: IGN_OUT -> IGN_IN
- J2 pad 2: ETB_OUT -> ETB_IN
- J2 pad 5: APPS1 -> APPS1_RAW
- J2 pad 6: APPS2 -> APPS2_RAW
- J2 pad 7: TPS1 -> TPS1_RAW
- J2 pad 8: TPS2 -> TPS2_RAW
- J5 pad A4: VBUS -> Net-(D10-A)
- J5 pad A9: VBUS -> Net-(D10-A)
- J5 pad B4: VBUS -> Net-(D10-A)
- J5 pad B9: VBUS -> Net-(D10-A)
- Q1 pad 2: IGN_OUT -> GND
- Q1 pad 3: +12V -> IGN_IN
- Q2 pad 2: ETB_OUT -> GND
- Q2 pad 3: +12V -> ETB_IN
- R10 pad 1: Net-(R10-Pad1) -> /PG
- R10 pad 2: IGN_OUT -> /buckVCC
- R11 pad 1: IGN_IND -> Net-(D11-A)
- R11 pad 2: Net-(R10-Pad1) -> /FB
- R12 pad 1: GND -> /FB
- R12 pad 2: IGN_IND -> GND
- R8 pad 1: Net-(R8-Pad1) -> Net-(D1-A)
- R8 pad 2: Net-(D1-A) -> GND
- U2 pad 10: unconnected-(U2-PA0-Pad10) -> APPS1
- U2 pad 11: unconnected-(U2-PA1-Pad11) -> APPS2
- U2 pad 12: unconnected-(U2-PA2-Pad12) -> TPS1
- U2 pad 13: unconnected-(U2-PA3-Pad13) -> TPS2
- U2 pad 40: APPS1 -> unconnected-(U2-PB4-Pad40)
- U2 pad 41: APPS2 -> unconnected-(U2-PB5-Pad41)
- U2 pad 42: TPS1 -> unconnected-(U2-PB6-Pad42)
- U2 pad 43: TPS2 -> unconnected-(U2-PB7-Pad43)
- U2 pad 5: unconnected-(U2-PF0-Pad5) -> CYST_IN
- U2 pad 6: unconnected-(U2-PF1-Pad6) -> CYST_OUT
- U3 pad 5: VBUS -> Net-(D10-A)
- U5 pad 1: IGN_IND -> Net-(U5A--)
- U5 pad 2: GND -> Net-(U5A--)
- U5 pad 3: ETB_IND -> Net-(U5A-+)
- U5 pad 4: Net-(R13-Pad1) -> Earth
- U5 pad 5: +3V3 -> Net-(U5B-+)
- U5 pad 6: Net-(R8-Pad1) -> Net-(U5B--)
