File: apppd.kicad_sch (KiCad schematic)
At the start: 99 parts, among them J1 Conn_SWD, J2 APPPD Connector, J4 2601-1102, J5 USB_C_Receptacle_USB2.0_16P, Q1 AO3400A, Q2 AO3400A, Q3 PMV100EPA, SW1 NRST, SW2 BOOT0, U1 AP2112K-3.3, U2 STM32F072CBTx, U3 USBLC6-2SC6, U4 TCAN337, U5 TLV9062xD, U6 LMR33610ADDAR, U7 TLV9062xD, Y1 ABM8AIG-24.000MHz-8-2Z-T

Commit message: Fixed ERC power warnings, AQ1005 ratings, and mounting holes
Cleaned up ERC to 0 errors/0 warnings, fixed the AQ1005 TVS description to match the datasheet, and added the missing mounting holes to the schematic.
Parts:
- added H1, H2, H3, H4: MountingHole_Pad, symbol Mechanical:MountingHole_Pad
- J4: symbol telemetry:2601-1102 -> apppd:2601-1102
- SW1, SW2: symbol EasyEDA:TS-1088-AR02016 -> apppd:TS-1088-AR02016
- Y1: symbol telemetry:ABM8AIG-24.000MHz-8-2Z-T -> apppd:ABM8AIG-24.000MHz-8-2Z-T
Connections:
- net GND: now also H1.1, H2.1, H3.1, H4.1

Commit message: Swapped inductor due to availability
Parts:
- L1: footprint Inductor_SMD:L_Vishay_IHLP-1616 -> Inductor_SMD:L_Vishay_IHLP-2525
